File: reactor/ESP32/pwm/pcb/v400/BioReactify/BioReactify.kicad_pcb (KiCad board)
At the start: 4 copper layers, 100 x 100 mm, 106 parts, among them IC3 MJ5688-B111-HR1-C, IC4 MJ5688-B111-HR1-C, J1 Conn_01x02, J10 Conn_01x06_Pin, J11 Conn_01x04_Pin, J12 Conn_01x04_Pin, J13 Conn_01x04_Pin, J14 Conn_01x04_Pin, J15 KF25C-7.62-2P, J16 KF25C-7.62-2P, J17 Conn_01x04_Pin, J18 Conn_01x02, J19 Conn_01x02, J2 Conn_01x02, J20 Conn_01x02, J21 Conn_01x02, J22 Conn_01x02, J23 Conn_01x02, J3 Conn_01x02, J4 Conn_01x02, J5 Conn_01x02, J6 Conn_01x02, J7 Conn_01x02, J8 Conn_01x02, J9 Conn_01x06_Pin, Q1 IRLZ44N, Q2 IRLZ44N, Q3 IRLZ44N, Q4 IRLZ44N, Q5 IRLZ44N, Q6 IRLZ44N, SW1 SW_DIP_x08, SW2 SW_DIP_x01, U1 LD1117S33TR_SOT223, U10 4N25, U11 4N25, U12 4N25, U13 MAX3490xSA, U2 MCP3208, U3 TCA9544A, U5 ESP32-DEVKIT-V1, U6 ACS712xLCBTR-030B3, U7 4N25, U8 4N25, U9 4N25

Commit message: espnow prototype
Parts:
- moved D6 0.95 mm to (189.8, 137.4)
Routing:
- net +3.3V: track 79.4 -> 364.1 mm, vias 15 -> 14
- net +12V: track 164.5 -> 290.8 mm
- net /PQ4: track 24.7 -> 32.7 mm
- net /CS3: track 91.5 -> 93.6 mm, vias 0 -> 2
- net /FETNEG0: track 132.1 -> 134.2 mm
- net -12V: track 14.7 -> 16.0 mm, vias 11 -> 7
- net /CH4: track 40.9 -> 40.3 mm
- net /CH3: track 107.2 -> 106.7 mm
- net /CS2: track 81.6 -> 81.8 mm, vias 0 -> 2
- net GND: vias 31 -> 28
- removed copper zone on B.Cu, net +12V
- removed copper zone on B.Cu, net +3.3V
- removed copper zone on F.Cu, net -12V

Commit message: Output class in cpp; Connect 2 boards to 1 experiment
Parts:
- added C10: 10uf, Capacitor_SMD:C_0603_1608Metric, B.Cu at (124.8, 90.8)
- added C11: 10uf, Capacitor_SMD:C_0603_1608Metric, B.Cu at (124.7, 93.2)
- added C12: 10uf, Capacitor_SMD:C_0603_1608Metric, B.Cu at (124.7, 95.8)
- added C13: 10uf, Capacitor_SMD:C_0603_1608Metric, B.Cu at (124.7, 98.3)
- added C14: 10uf, Capacitor_SMD:C_0603_1608Metric, B.Cu at (124.7, 100.8)
- added C5: 10uf, Capacitor_SMD:C_0603_1608Metric, B.Cu at (124.8, 83.2)
- added C8: 10uf, Capacitor_SMD:C_0603_1608Metric, B.Cu at (124.8, 85.8)
- added C9: 10uf, Capacitor_SMD:C_0603_1608Metric, B.Cu at (124.8, 88.2)
- J11, J12, J13, J14: footprint Connector_Phoenix_MC:PhoenixContact_MCV_1,5_4-G-3.81_1x04_P3.81mm_Vertical -> Connector_JST:JST_PH_B4B-PH-K_1x04_P2.00mm_Vertical
- moved J14 9.08 mm to (152.8, 126.0)
- moved J13 8.07 mm to (152.8, 120.0)
- moved J11 7.91 mm to (152.8, 108.0)
- moved J12 7.66 mm to (152.8, 114.0)
- moved J17 1.20 mm to (159.3, 100.5)
Routing:
- net /i2c/SD1: track 45.7 -> 70.6 mm
- net /i2c/SC3: track 67.4 -> 54.5 mm
- net /i2c/SC2: track 61.1 -> 49.6 mm
- net /i2c/SC1: track 55.9 -> 46.0 mm
- net /i2c/SD3: track 59.3 -> 51.2 mm
- net /i2c/SD2: track 54.4 -> 47.9 mm
- net /i2c/SC0: track 42.4 -> 39.1 mm
- net GND: track 64.6 -> 67.3 mm, vias 28 -> 36
- net /CH1: track 71.9 -> 74.1 mm
- net /CH2: track 89.4 -> 91.6 mm
- net /CH7: track 53.6 -> 55.8 mm
- net /CH3: track 106.7 -> 108.9 mm
- net /CH6: track 43.9 -> 46.1 mm
- net /CH5: track 39.2 -> 41.4 mm
- net /CH4: track 40.3 -> 42.5 mm
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
Commit message: update pcb: incomplete
Parts:
- removed C3: 10uF, Capacitor_SMD:C_0805_2012Metric
- removed J15: KF25C-7.62-2P, SamacSys_Parts:KF25C7622P
- removed J8: Conn_01x02, Connector_Phoenix_MC:PhoenixContact_MCV_1,5_2-G-3.81_1x02_P3.81mm_Vertical
- removed SW1: SW_DIP_x08, Button_Switch_SMD:SW_DIP_SPSTx08_Slide_6.7x21.88mm_W8.61mm_P2.54mm_LowProfile
- removed SW2: SW_DIP_x01, Button_Switch_SMD:SW_DIP_SPSTx01_Slide_6.7x4.1mm_W8.61mm_P2.54mm_LowProfile
- added C15: 10uF, Capacitor_SMD:C_0805_2012Metric, F.Cu at (128.7, 119.4)
- added C16: 0.1uF, Capacitor_SMD:C_0603_1608Metric_Pad1.08x0.95mm_HandSolder, F.Cu at (111.1, 121.8)
- added C17: 0.1uF, Capacitor_SMD:C_0603_1608Metric_Pad1.08x0.95mm_HandSolder, F.Cu at (111.6, 132.9)
- added C18: 0.1uF, Capacitor_SMD:C_0603_1608Metric_Pad1.08x0.95mm_HandSolder, F.Cu at (111.4, 144.1)
- added C19: 0.1uF, Capacitor_SMD:C_0603_1608Metric_Pad1.08x0.95mm_HandSolder, F.Cu at (117.4, 149.2)
- added C20: 0.1uF, Capacitor_SMD:C_0603_1608Metric_Pad1.08x0.95mm_HandSolder, F.Cu at (128.9, 149.1)
- added R41: 3.4K, Resistor_SMD:R_0603_1608Metric_Pad0.98x0.95mm_HandSolder, F.Cu at (144.7, 152.6)
- added R42: 150, Resistor_SMD:R_0603_1608Metric_Pad0.98x0.95mm_HandSolder, F.Cu at (106.5, 133.1)
- added R43: 3.4K, Resistor_SMD:R_0603_1608Metric_Pad0.98x0.95mm_HandSolder, F.Cu at (112.3, 146.7)
- added R44: 3.4K, Resistor_SMD:R_0603_1608Metric_Pad0.98x0.95mm_HandSolder, F.Cu at (155.8, 152.7)
- added R45: 7.8K, Resistor_SMD:R_0603_1608Metric_Pad0.98x0.95mm_HandSolder, F.Cu at (129.2, 154.0)
- added R46: 4.1K, Resistor_SMD:R_0603_1608Metric_Pad0.98x0.95mm_HandSolder, F.Cu at (134.6, 151.5)
- added R47: 4.1K, Resistor_SMD:R_0603_1608Metric_Pad0.98x0.95mm_HandSolder, F.Cu at (136.1, 151.5)
- added R48: 1.5K, Resistor_SMD:R_0603_1608Metric_Pad0.98x0.95mm_HandSolder, F.Cu at (133.0, 151.5)
- added R49: 150, Resistor_SMD:R_0603_1608Metric_Pad0.98x0.95mm_HandSolder, F.Cu at (106.4, 144.2)
- added R50: 3.4K, Resistor_SMD:R_0603_1608Metric_Pad0.98x0.95mm_HandSolder, F.Cu at (120.0, 148.3)
- added U14: TLV9001IDCK, Package_TO_SOT_SMD:SOT-353_SC-70-5, F.Cu at (109.0, 134.6)
- added U15: TLV9001IDCK, Package_TO_SOT_SMD:SOT-353_SC-70-5, F.Cu at (130.7, 151.6)
- added U16: TLV9001IDCK, Package_TO_SOT_SMD:SOT-353_SC-70-5, F.Cu at (108.8, 145.8)
- added U17: LD1117S33TR_SOT223, Package_TO_SOT_SMD:SOT-223-3_TabPin2, F.Cu at (120.3, 116.2)
- added U18: MCP3208, Package_DIP:DIP-16_W7.62mm_Socket, F.Cu at (127.8, 129.9)
- added U4: TLV9001IDCK, Package_TO_SOT_SMD:SOT-353_SC-70-5, F.Cu at (119.2, 151.7)
- C10, C11, C12, C13, C5, C8, C9: value 10uf -> 0.047uf; moved to F.Cu
- C14: value 10uf -> 100nF; footprint Capacitor_SMD:C_0603_1608Metric -> Capacitor_SMD:C_0805_2012Metric; moved to F.Cu
- J5, J6, J7: footprint Connector_Phoenix_MC:PhoenixContact_MCV_1,5_2-G-3.81_1x02_P3.81mm_Vertical -> Connector_Phoenix_MC:PhoenixContact_MC_1,5_2-G-3.81_1x02_P3.81mm_Horizontal
- R13: footprint Resistor_SMD:R_0805_2012Metric -> Resistor_SMD:R_0603_1608Metric_Pad0.98x0.95mm_HandSolder
- R14, R20: value 10K -> 3.4K; footprint Resistor_SMD:R_0805_2012Metric -> Resistor_SMD:R_0603_1608Metric_Pad0.98x0.95mm_HandSolder
- R15: value 150 -> 3.4K; footprint Resistor_SMD:R_0805_2012Metric -> Resistor_SMD:R_0603_1608Metric_Pad0.98x0.95mm_HandSolder
- R16: value 10K -> 7.8K; footprint Resistor_SMD:R_0805_2012Metric -> Resistor_SMD:R_0603_1608Metric_Pad0.98x0.95mm_HandSolder
- R17: value 150 -> 4.1K; footprint Resistor_SMD:R_0805_2012Metric -> Resistor_SMD:R_0603_1608Metric_Pad0.98x0.95mm_HandSolder
- R18: value 10K -> 4.1K; footprint Resistor_SMD:R_0805_2012Metric -> Resistor_SMD:R_0603_1608Metric_Pad0.98x0.95mm_HandSolder
- R19: value 10K -> 1.5K; footprint Resistor_SMD:R_0805_2012Metric -> Resistor_SMD:R_0603_1608Metric_Pad0.98x0.95mm_HandSolder
- U2: value MCP3208 -> TLV9001IDCK; footprint Package_DIP:DIP-16_W7.62mm_Socket -> Package_TO_SOT_SMD:SOT-353_SC-70-5
- moved J18 107.4 mm to (207.6, 65.1), turned to 90 degrees
- moved J19 88.4 mm to (207.7, 82.1), turned to 90 degrees
- moved J20 69.7 mm to (207.7, 99.0), turned to 90 degrees
- moved J10 58.3 mm to (102.6, 91.3), turned to 0 degrees
- moved J7 55.0 mm to (155.7, 157.4), turned to 0 degrees
- moved J5 53.4 mm to (130.7, 157.4), turned to 0 degrees
- moved J6 52.8 mm to (144.7, 157.3), turned to 0 degrees
- moved J9 52.6 mm to (108.5, 91.3), turned to 0 degrees
- moved J21 51.7 mm to (207.7, 115.6), turned to 90 degrees
- moved D9 51.5 mm to (173.3, 60.8)
- moved C5 50.8 mm to (130.3, 133.8), turned to -90 degrees
- moved C8 50.5 mm to (140.5, 133.8), turned to -90 degrees
- moved R23 47.5 mm to (173.3, 63.1), turned to 0 degrees
- moved C10 46.8 mm to (143.0, 133.8), turned to -90 degrees
- moved C9 46.2 mm to (132.8, 133.8), turned to -90 degrees
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Connections:
- C10 pad 1: GND -> /adc0/CH6
- C10 pad 2: /CH3 -> GND
- C11 pad 1: /CH4 -> /adc0/CH3
- C12 pad 1: /CH5 -> /adc0/CH7
- C13 pad 1: /CH6 -> /adc0/CH4
- C14 pad 1: /CH7 -> /5v_protected
- C5 pad 1: GND -> /adc0/CH1
- C5 pad 2: /CH0 -> GND
- C8 pad 1: GND -> /adc0/CH5
- C8 pad 2: /CH1 -> GND
- C9 pad 1: GND -> /adc0/CH2
- C9 pad 2: /CH2 -> GND
- J1 pad 1: /CH0 -> /adc0/IN1
- J11 pad 3: +3.3V -> GND
- J11 pad 4: GND -> +3.3V
- J12 pad 3: +3.3V -> GND
- J12 pad 4: GND -> +3.3V
- J13 pad 3: +3.3V -> GND
- J13 pad 4: GND -> +3.3V
- J14 pad 3: +3.3V -> GND
- J14 pad 4: GND -> +3.3V
- J2 pad 1: /CH1 -> /adc0/IN2
- J3 pad 1: /CH2 -> /adc0/IN3
- J4 pad 1: /CH3 -> +3.3VADC
- J4 pad 2: GND -> /adc0/IN4
- J5 pad 1: /CH4 -> +3.3VADC
- J5 pad 2: GND -> /adc0/IN5
- J6 pad 1: /CH5 -> /adc0/IN6
- J7 pad 1: /CH6 -> /adc0/IN7
- R13 pad 2: /analogs/ACH0 -> /adc0/IN1
- R14 pad 1: +3.3V -> /adc0/CH1
- R14 pad 2: /analogs/ACH4 -> /adc0/ICH1
- R15 pad 1: GND -> /adc0/CH5
- R15 pad 2: /analogs/ACH1 -> /adc0/TCH5
- R16 pad 1: +3.3V -> GND
- R16 pad 2: /analogs/ACH5 -> /adc0/IN4
- R17 pad 1: GND -> Net-(U4--)
- R17 pad 2: /analogs/ACH2 -> +3.3VADC
- R18 pad 1: +3.3V -> GND
- R18 pad 2: /analogs/ACH6 -> Net-(U4--)
- R19 pad 1: +3.3V -> Net-(U4--)
- R19 pad 2: /analogs/ACH3 -> /adc0/TCH4
- R20 pad 1: +3.3V -> /adc0/CH2
- R20 pad 2: /analogs/ACH7 -> /adc0/ICH2
- U2 pad 1: /CH0 -> /adc0/IN1
- U2 pad 2: /CH1 -> GND
- U2 pad 3: /CH2 -> /adc0/ICH1
- U2 pad 4: /CH3 -> /adc0/ICH1
- U2 pad 5: /CH4 -> +3.3VADC
- U6 pad 7: Net-(U6-VIOUT) -> /CH0
Routing:
- net +3.3V: track 362.1 -> 0.00 mm, vias 14 -> 0
- net /FETNEG0: track 134.2 -> 21.3 mm
- net /CH3: track 108.9 -> 0.00 mm
- net /CH0: track 102.2 -> 0.00 mm, vias 1 -> 0
- net /CH2: track 91.6 -> 0.00 mm
- net /FETNEG1: track 112.9 -> 21.4 mm
- net +12V: track 290.8 -> 199.9 mm
- net /CH1: track 74.1 -> 0.00 mm
- net /FETNEG2: track 89.5 -> 21.4 mm
- net GND: track 67.3 -> 0.00 mm, vias 36 -> 1
- net /CH7: track 55.8 -> 0.00 mm
- net Net-(U6-VIOUT): track 47.1 -> 0.00 mm
- net /CH6: track 46.1 -> 0.00 mm
- net /FETNEG3: track 64.6 -> 21.7 mm
- net /CH4: track 42.5 -> 0.00 mm
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- added copper zone on B.Cu, net +12V
- added copper zone on F.Cu, net -12V
- removed copper zone on F.Cu, net GND
- removed copper zone on In1.Cu, net GND
- removed copper zone on In2.Cu, net GND
Other:
- board size 100 x 100 mm -> 110 x 110 mm
