File: reactor/ESP32/pwm/pcb/v400/BioReactify/adc0.kicad_sch (KiCad schematic)
At the start: 46 parts, among them J1 Conn_01x02, J2 Conn_01x02, J3 Conn_01x02, J4 Conn_01x02, J5 Conn_01x02, J6 Conn_01x02, J7 Conn_01x02, U14 TLV9001IDCK, U15 TLV9001IDCK, U16 TLV9001IDCK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

Commit message: update pcb: incomplete
Parts:
- J6, J7: footprint Connector_Phoenix_MC:PhoenixContact_MCV_1,5_2-G-3.81_1x02_P3.81mm_Vertical -> Connector_Phoenix_MC:PhoenixContact_MC_1,5_2-G-3.81_1x02_P3.81mm_Horizontal
Connections:
- net +3.3V is gone; now on net +3.3VADC: R17.2, R46.2
Other:
- note added: "@3.4K input impedance Max Clock speed < 1MHz"
- note added: "Vishay NTCLE413 10K 1% Temperature swing: 0oC - 70oC Gain = ( (R17||R18) + R19 ) / (R17||R18) Gain = 1.73"
- note removed: "@ 3.4K input impedance Max Clock speed < 1MHz"
- note removed: "Vishay NTCLE413 10K 1% Temperature swing: 0oC - 70oC Gain = 1.73"
- title: BioReactify Master -> (none)
