File: hardware/BioReactify/adc0.kicad_sch (KiCad schematic)
At the start: 46 parts, among them J1 Conn_01x02, J2 Conn_01x02, J3 Conn_01x02, J4 Conn_01x02, J5 Conn_01x02, J6 Conn_01x02, J7 Conn_01x02, U14 TLV9001IDCK, U15 TLV9001IDCK, U16 TLV9001IDCK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

Commit message: PCB complete, biomass sensor PCB complete
Parts:
- removed J6, J7: Conn_01x02, Connector_Phoenix_MC:PhoenixContact_MC_1,5_2-G-3.81_1x02_P3.81mm_Horizontal, symbol Connector_Generic:Conn_01x02
- added J6, J7: Conn_01x03, Connector_Phoenix_MC:PhoenixContact_MC_1,5_3-G-3.81_1x03_P3.81mm_Horizontal, symbol Connector_Generic:Conn_01x03
- added TP3: TestPoint, TestPoint:TestPoint_Pad_1.0x1.0mm, symbol Connector:TestPoint
- R14, R15, R20, R41, R43, R44, R50: value 3.4K -> 1K
Connections:
- net +3.3VADC: now also J6.1 (Pin_1), J7.1 (Pin_1), TP3.1
- net GND: now also J6.2 (Pin_2), J7.2 (Pin_2)
- net ICH3: now also U2.3 (-), U2.4; no longer U16.3 (-), U16.4
- net IN6: now also J6.3 (Pin_3)
- net IN7: now also J7.3 (Pin_3)
- net 5v_protected renamed +5V
- removed net ICH1: R14.2, U2.3 (-), U2.4
- net ICH2 renamed ICH4
- net ICH4: now also R50.2; no longer R20.2
- net TCH4 renamed TCH1
- net TCH1: now also R14.2; no longer R50.2
- net TCH5 renamed TCH2
- net TCH2: now also R20.2; no longer R15.2
- new net ICH5: R15.2, U16.3 (-), U16.4
Other:
- note added: "@1K input impedance Max Clock speed < 2MHz"
- note added: "Max sampling rate tacq_min = (R*(C+Cin)*ln(Cin*2^(n+1)/(C+Cin))) = 9.34us tconv = 12 * Clock_cycle = 6us sampling_rate = 1 / (tacq_min + tconv) = 65KHz"
- note added: "RC filter fc = 1 / 2piRC fc = 3386Hz"
- note added: "Target Sampling rate 2.2KHz"
- note added: "Vishay NTCLE413 10K 1% Temperature swing: 0oC - 70oC Gain = ( (R17||R18) + R19 ) / (R17||R18) = 1.73 Vout = Vcc * ( R16 / (Rnt + R16) ) * Gain - ( Vcc * R19 / R17) K = (1 / Gain) * ( Vout / Vcc + R19 / R17) Rntc = R16 * (1 / K - 1)"
- note removed: "@3.4K input impedance Max Clock speed < 1MHz"
- note removed: "Max sampling rate 1 / (R*(C+Cin)*ln(Cin*2^(n+1)/(C+Cin))) = 31kHz"
- note removed: "RC filter fc = 1 / 2piRC fc = 995Hz"
- note removed: "Target Sampling rate 2.0KHz"
- note removed: "Vishay NTCLE413 10K 1% Temperature swing: 0oC - 70oC Gain = ( (R17||R18) + R19 ) / (R17||R18) Gain = 1.73"
- moved on the sheet: R16, R17, R18, R19, R45, R46, R47, R48, U15, U4
