File: hardware/BioReactify/BioReactify.kicad_sch (KiCad schematic)
At the start: 65 parts, among them IC3 MJ5688-B111-HR1-C, IC4 MJ5688-B111-HR1-C, J10 Conn_01x06_Pin, J16 KF25C-7.62-2P, J17 Conn_01x04_Pin, J18 Conn_01x02, J19 Conn_01x02, J20 Conn_01x02, J21 Conn_01x02, J22 Conn_01x02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

Commit message: PCB complete, biomass sensor PCB complete
Parts:
- removed D11: LED, LED_SMD:LED_0805_2012Metric, symbol Device:LED
- removed D6: 50V 5A, Diode_SMD:D_SMA, symbol Device:D
- removed D8: 5.1V, Diode_SMD:D_SMB, symbol Device:D_Zener
- removed IC3: MJ5688-B111-HR1-C, SamacSys_Parts:MJ5688B111HR1C, symbol SamacSys_Parts:MJ5688-B111-HR1-C
- removed J17: Conn_01x04_Pin, Connector_PinHeader_2.54mm:PinHeader_1x04_P2.54mm_Vertical, symbol Connector:Conn_01x04_Pin
- removed Q6: IRLZ44N, Package_TO_SOT_THT:TO-220-3_Vertical, symbol Transistor_FET:IRLZ44N
- removed R11: 100, Resistor_SMD:R_0805_2012Metric, symbol Device:R_US
- removed R12: 470, Resistor_SMD:R_0805_2012Metric, symbol Device:R_US
- removed R25: 550, Resistor_SMD:R_0805_2012Metric, symbol Device:R_US
- removed U12: 4N25, Package_DIP:DIP-6_W7.62mm_Socket, symbol Isolator:4N25
- added C21: 10uF, Capacitor_SMD:C_0805_2012Metric, symbol Device:C_Small
- added C3: 100nF, Capacitor_SMD:C_0805_2012Metric, symbol Device:C_Small
- added D6: VS12VBA1HS, Diode_SMD:D_0603_1608Metric_Pad1.05x0.95mm_HandSolder, symbol Device:D_Zener
- added J17, J8: Conn_01x02, Connector_Phoenix_MC:PhoenixContact_MC_1,5_2-G-3.81_1x02_P3.81mm_Horizontal, symbol Connector_Generic:Conn_01x02
- added J24: Conn_01x03, Connector_Phoenix_MC:PhoenixContact_MC_1,5_3-G-3.81_1x03_P3.81mm_Horizontal, symbol Connector_Generic:Conn_01x03
- added TP1, TP2: TestPoint, TestPoint:TestPoint_Pad_1.0x1.0mm, symbol Connector:TestPoint
- added U12: LD1117S50TR_SOT223, Package_TO_SOT_SMD:SOT-223-3_TabPin2, symbol Regulator_Linear:LD1117S50TR_SOT223
- D7: value 50V 2A -> B340A-13-F; footprint Diode_SMD:D_SMB -> Diode_SMD:D_SMA
- F1: value 6V 1.5A -> 13.2V 3A
Connections:
- net D33 is gone; now on net Q4: U5.22 (D33)
- net FETNEG5 is gone; now on net GND: J23.1 (Pin_1)
- net +12V: no longer J23.2 (Pin_2)
- net +3.3V: now also TP2.1
- net +5V: now also C1.1, J23.2 (Pin_2), U1.3 (VI), C21.1, TP1.1, U12.2 (VO); no longer F1.1
- net 5v_protected: no longer C1.1, D7.1 (K), U1.3 (VI)
- net GND: now also C21.2, C3.2, D6.2 (A), J17.1 (Pin_1), J8.1 (Pin_1), U12.1 (GND)
- net Q4: no longer U5.24 (D26)
- net SPI_DIN: now also U5.9 (D18)
- net SPI_DOUT: no longer U5.9 (D18)
- net -12V renamed GNDPWR
- net D32 renamed PIN32
- net PIN32: now also J24.1 (Pin_1)
- net D34: no longer names the net of U5.20 (D35)
- net D35: no longer names the net of U5.19 (D34)
- net Q5 renamed DAC1
- net DAC1: now also J24.2 (Pin_2)
- net fuse_5v: no longer names the net of D7.2 (A), F1.2
- new net DAC2: J24.3 (Pin_3), U5.24 (D26)
- new net VCC: D6.1 (K), F1.1, J17.2 (Pin_2), J8.2 (Pin_2)
- new net Vcc_protected: C3.1, D7.1 (K), U12.3 (VI)
- no-connect marks 20 -> 17
Other:
- note added: "+9V < Vcc < +12V"
- moved on the sheet: C1, C2, C4, C6, C7, D2, D4, D7, D9, F1, H1, H2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

Commit message: Hardware updated
Parts:
- removed C1, C3: 100nF, Capacitor_SMD:C_0805_2012Metric, symbol Device:C_Small
- removed C2, C21, C4, C6, C7: 10uF, Capacitor_SMD:C_0805_2012Metric, symbol Device:C_Small
- removed D1, D2, D3, D4, D5: 50V 5A, Diode_SMD:D_SMA, symbol Device:D
- removed D6: VS12VBA1HS, Diode_SMD:D_0603_1608Metric_Pad1.05x0.95mm_HandSolder, symbol Device:D_Zener
- removed D7: B340A-13-F, Diode_SMD:D_SMA, symbol Device:D
- removed D9: LED, LED_SMD:LED_0805_2012Metric, symbol Device:LED
- removed F1: 13.2V 3A, Fuse:Fuse_1206_3216Metric, symbol Device:Fuse
- removed IC4: MJ5688-B111-HR1-C, SamacSys_Parts:MJ5688B111HR1C, symbol SamacSys_Parts:MJ5688-B111-HR1-C
- removed J10, J9: Conn_01x06_Pin, Connector_PinHeader_2.54mm:PinHeader_1x06_P2.54mm_Vertical, symbol Connector:Conn_01x06_Pin
- removed J16: KF25C-7.62-2P, SamacSys_Parts:KF25C7622P, symbol SamacSys_Parts:KF25C-7.62-2P
- removed J17, J18, J19, J20, J21, J22, J23, J8: Conn_01x02, Connector_Phoenix_MC:PhoenixContact_MC_1,5_2-G-3.81_1x02_P3.81mm_Horizontal, symbol Connector_Generic:Conn_01x02
- removed J24: Conn_01x03, Connector_Phoenix_MC:PhoenixContact_MC_1,5_3-G-3.81_1x03_P3.81mm_Horizontal, symbol Connector_Generic:Conn_01x03
- removed Q1, Q2, Q3, Q4, Q5: IRLZ44N, Package_TO_SOT_THT:TO-220-3_Vertical, symbol Transistor_FET:IRLZ44N
- removed R1, R23, R3, R5, R7, R9: 100, Resistor_SMD:R_0805_2012Metric, symbol Device:R_US
- removed R10, R2, R4, R6, R8: 470, Resistor_SMD:R_0805_2012Metric, symbol Device:R_US
- removed R21: 0, Resistor_SMD:R_1206_3216Metric_Pad1.30x1.75mm_HandSolder, symbol Device:R_US
- removed R24: 10K, Resistor_SMD:R_0805_2012Metric, symbol Device:R_US
- removed R28: 120, Resistor_SMD:R_0603_1608Metric, symbol Device:R_US
- removed TP1, TP2: TestPoint, TestPoint:TestPoint_Pad_1.0x1.0mm, symbol Connector:TestPoint
- removed U1: LD1117S33TR_SOT223, Package_TO_SOT_SMD:SOT-223-3_TabPin2, symbol Regulator_Linear:LD1117S33TR_SOT223
- removed U10, U11, U7, U8, U9: 4N25, Package_DIP:DIP-6_W7.62mm_Socket, symbol Isolator:4N25
- removed U12: LD1117S50TR_SOT223, Package_TO_SOT_SMD:SOT-223-3_TabPin2, symbol Regulator_Linear:LD1117S50TR_SOT223
- removed U13: MAX3490xSA, Package_SO:SOIC-8_3.9x4.9mm_P1.27mm, symbol Interface_UART:MAX3490xSA
- removed U5: ESP32-DEVKIT-V1, other:MODULE_ESP32_DEVKIT_V1, symbol ESP32-DEVKIT-V1:ESP32-DEVKIT-V1
- removed U6: ACS712xLCBTR-030B3, Package_SO:SOIC-8_3.9x4.9mm_P1.27mm, symbol custom:ACS712xLCBTR-030B3
- added C12: 10uF, Capacitor_SMD:C_0805_2012Metric, symbol Device:C
- added J2: Conn_01x10_Pin, Connector_PinHeader_2.54mm:PinHeader_1x10_P2.54mm_Vertical, symbol Connector:Conn_01x10_Pin
- added J3: Micro_SD_Card, custom:TF-SMD_THD2528-11SD-GF, symbol Connector:Micro_SD_Card
- added J4: Conn_01x02_Pin, Connector_PinHeader_2.54mm:PinHeader_1x02_P2.54mm_Vertical, symbol Connector:Conn_01x02_Pin
- added R26, R27: 10K, Resistor_SMD:R_0805_2012Metric_Pad1.20x1.40mm_HandSolder, symbol Device:R_US
- added U1: ESP32-DEVKIT-V1, custom:MODULE_ESP32_DEVKIT_V1, symbol ESP32-DEVKIT-V1:ESP32-DEVKIT-V1
- H1, H2, H3, H4: footprint MountingHole:MountingHole_3.2mm_M3_ISO7380_Pad -> MountingHole:MountingHole_3.2mm_M3_DIN965_Pad_TopBottom
Connections:
- net CS1: now also J3.2 (DAT3/CD), R27.2, U1.3 (D15)
- net DAC1: now also J2.5 (Pin_5), U1.23 (D25)
- net DAC2: now also J2.6 (Pin_6), U1.24 (D26)
- net GND: now also H1.1, H2.1, H3.1, H4.1, C12.2, J3.6 (VSS), J4.2 (Pin_2), U1.2 (GND), U1.29 (GND)
- net SCL: now also U1.14 (D22)
- net SDA: now also U1.11 (D21)
- new net: J2.10 (Pin_10), U1.28 (D13)
- new net: J2.3 (Pin_3), U1.21 (D32)
- new net: J2.4 (Pin_4), U1.22 (D33)
- new net: J2.7 (Pin_7), U1.25 (D27)
- new net: J2.8 (Pin_8), U1.26 (D14)
- new net: J2.9 (Pin_9), U1.27 (D12)
- new net CS: R26.2, U1.15 (D23)
- new net D2: J2.2 (Pin_2), U1.20 (D35), U1.4 (D2)
- new net D4: J2.1 (Pin_1), U1.19 (D34), U1.5 (D4)
- new net MISO: J3.7 (DAT0), U1.9 (D18)
- new net MOSI: J3.3 (CMD), U1.10 (D19)
- new net RS485/RX2: U1.6 (RX2)
- new net RS485/TX2: U1.7 (TX2)
- new net SCLK: J3.5 (CLK), U1.8 (D5)
- new net VDD: C12.1, J3.4 (VDD), J4.1 (Pin_1), R26.1, R27.1, U1.1 (3V3)
- no-connect marks 17 -> 9
Other:
- removed sheet adc0
- removed sheet i2c
- added sheet ADC (ADC.kicad_sch)
- added sheet I2C (I2C.kicad_sch)
- added sheet RS485 (RS485.kicad_sch)
- note added: "VDD = +3.3V"
- note removed: "+9V < Vcc < +12V"
- note removed: "Analog Read"
- note removed: "Full Duplex RS485"
- note removed: "Power Stage"
- note removed: "Power Supply"
- note removed: "SPI"
- title: BioReactify Master -> (none)
