File: hardware/smart_sleeve/smart_sleeve.kicad_pcb (KiCad board)
At the start: 2 copper layers, 60 x 50 mm, 2 parts

Commit message: PCB complete, biomass sensor PCB complete
Parts:
- removed H1, H2: MountingHole_Pad, MountingHole:MountingHole_2.2mm_M2_Pad
- added J1: Conn_01x04_Pin, Connector_PinHeader_2.54mm:PinHeader_1x04_P2.54mm_Vertical, F.Cu at (156.3, 100.1)
- added J2: Screw_Terminal_01x02, TerminalBlock_Phoenix:TerminalBlock_Phoenix_PT-1,5-2-5.0-H_1x02_P5.00mm_Horizontal, F.Cu at (154.6, 119.1)
- added J3: Conn_01x02_Pin, Connector_PinHeader_2.54mm:PinHeader_1x02_P2.54mm_Vertical, F.Cu at (156.5, 84.5)
- added TH1: 10K, Resistor_THT:R_Axial_DIN0204_L3.6mm_D1.6mm_P1.90mm_Vertical, F.Cu at (175.2, 89.7)
Routing:
- net +3.3V: track 0.00 -> 20.9 mm
- net /Tout: track 0.00 -> 19.1 mm
- net /MOT_POS: track 0.00 -> 17.5 mm
- net /resistance: track 892.1 -> 902.1 mm
- net /MOT_NEG: track 0.00 -> 7.02 mm
Other:
- outline, holes or cut-outs redrawn
- board text added: "3.3V"
- board text added: "H0"
- board text added: "H1"
- board text added: "M+"
- board text added: "M-"
- board text added: "Tout"
