File: hardware/kicad/heating_element/heating_element.kicad_pcb (KiCad board)
At the start: 2 copper layers, 60 x 50 mm, 4 parts, among them J1 Conn_01x04_Pin, J2 Screw_Terminal_01x02, J3 Conn_01x02_Pin

Commit message: bug fix; reactor board update;
Parts:
- moved J3 36.4 mm to (190.0, 70.3), turned to 180 degrees
- moved J1 30.4 mm to (130.8, 83.6)
- moved J2 30.4 mm to (129.1, 102.6)
- moved TH1 30.4 mm to (149.7, 73.2)
Routing:
- net /Tout: track 19.1 -> 46.3 mm
- net +3.3V: track 20.9 -> 41.5 mm
Other:
- board size 60 x 50 mm -> 70 x 50 mm
