File: hardware/kicad/reactor/analog_input.kicad_sch (KiCad schematic)
At the start: 35 parts, among them J201 Conn_01x02_Pin, J202 Conn_01x02_Pin, J203 Conn_01x02_Pin, J204 Conn_01x02_Pin, J205 Conn_01x02_Pin, J206 Conn_01x03_Pin, J207 Conn_01x03_Pin, U201 TLV9001IDCK, U202 TLV9001IDCK, U203 TLV9001IDCK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

Commit message: bug fix; reactor board update;
Parts:
- R201, R205: value 7.8K -> 7.68K
- R202, R203, R206, R207: value 4.1K -> 4.3K
Changed lines of the file:
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@@
 			)
 		)
-		(property "Value" "7.8K"
+		(property "Value" "7.68K"
 			(at 22.098 60.96 0)
 			(effects
@@
 			)
 		)
-		(property "Value" "4.1K"
+		(property "Value" "4.3K"
 			(at 37.338 122.682 0)
 			(effects
@@
 			)
 		)
-		(property "Value" "4.1K"
+		(property "Value" "4.3K"
 			(at 37.338 132.588 0)
 			(effects
@@
 			)
 		)
-		(property "Value" "4.1K"
+		(property "Value" "4.3K"
 			(at 37.338 66.802 0)
 			(effects
@@
 			)
 		)
-		(property "Value" "7.8K"
+		(property "Value" "7.68K"
 			(at 22.098 116.84 0)
 			(effects
@@
 			)
 		)
-		(property "Value" "4.1K"
+		(property "Value" "4.3K"
 			(at 37.338 76.708 0)
 			(effects
