File: hardware/kicad/reactor/reactor.kicad_pcb (KiCad board)
At the start: 2 copper layers, 145 x 100 mm, 93 parts, among them J1 Conn_01x02_Pin, J2 Conn_01x02_Pin, J201 Conn_01x02_Pin, J202 Conn_01x02_Pin, J203 Conn_01x02_Pin, J204 Conn_01x02_Pin, J205 Conn_01x02_Pin, J206 Conn_01x03_Pin, J207 Conn_01x03_Pin, J3 Conn_01x02_Pin, J301 Conn_01x02, J302 Conn_01x02, J303 Conn_01x02, J304 Conn_01x02, J305 Conn_01x02, J4 Conn_02x09_Odd_Even, J5 Conn_01x02_Pin, J6 Conn_01x10, J7 Conn_01x03, Q301 IRLZ44N, Q302 IRLZ44N, Q303 IRLZ44N, Q304 IRLZ44N, Q305 IRLZ44N, U1 LD1117S50TR, U2 LD1117S33TR, U201 TLV9001IDCK, U202 TLV9001IDCK, U203 TLV9001IDCK, U204 TLV9001IDCK, U205 TLV9001IDCK, U3 LD1117S33TR, U301 4N25, U302 4N25, U303 4N25, U304 4N25, U305 4N25

Commit message: bug fix; reactor board update;
Parts:
- added D4: 50V 5A, Diode_SMD:D_SMA, F.Cu at (125.2, 43.4)
- added D5: 50V 5A, Diode_SMD:D_SMA, F.Cu at (116.0, 53.5)
- C1: value 0.1uF -> 0.22uF; footprint Capacitor_SMD:CP_Elec_4x5.4 -> Capacitor_SMD:C_0805_2012Metric_Pad1.18x1.45mm_HandSolder
- C2, C4, C6: value 10uF -> 0.1uF; footprint Capacitor_SMD:CP_Elec_4x5.3 -> Capacitor_SMD:C_1206_3216Metric
- C3, C5: footprint Capacitor_SMD:CP_Elec_4x5.4 -> Capacitor_SMD:C_1206_3216Metric
- R201, R205: value 7.8K -> 7.68K
- R202, R203, R206, R207: value 4.1K -> 4.3K
- U1: value LD1117S50TR -> LM340MPX-5.0/NOPB
- U2, U3: value LD1117S33TR -> TLV75733PDBV; footprint Package_TO_SOT_SMD:SOT-223-3_TabPin2 -> Package_TO_SOT_SMD:SOT-23-5
- moved D3 12.5 mm to (223.4, 41.9), turned to 180 degrees
- moved C4 12.0 mm to (129.0, 47.8), turned to -90 degrees
- moved C6 11.9 mm to (120.0, 57.7), turned to -90 degrees
- moved C2 11.6 mm to (106.4, 48.6)
- moved U3 9.07 mm to (115.9, 57.6), turned to 0 degrees
- moved C1 8.81 mm to (110.8, 42.3), turned to 0 degrees
- moved J3 8.22 mm to (219.5, 35.5), turned to 0 degrees
- moved C5 6.38 mm to (111.8, 57.7)
- moved J1 6.10 mm to (123.5, 34.0)
- moved D1 5.92 mm to (122.8, 39.1)
- moved D2 5.92 mm to (111.7, 39.1)
- moved F1 5.92 mm to (118.2, 39.1)
- moved D207 4.80 mm to (146.2, 117.2)
- moved U2 4.55 mm to (125.2, 47.7)
- moved D206 4.36 mm to (131.3, 117.4)
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Connections:
- J3 pad 1: +12V -> GNDPWR
- J3 pad 2: GNDPWR -> +12V
- U2 pad 1: GND -> +5V
- U2 pad 2: +3.3V -> GND
- U3 pad 1: GND -> +5V
- U3 pad 2: +3.3VADC -> GND
Routing:
- net +3.3VADC: track 376.2 -> 325.1 mm
- net +12V: track 249.6 -> 219.6 mm
- net +5V: track 50.8 -> 23.2 mm, vias 0 -> 4
- net +3.3V: track 19.2 -> 0.01 mm
- net GNDPWR: track 170.8 -> 163.8 mm, vias 1 -> 0
- net GND: track 76.7 -> 83.0 mm
- net /Vcc_protected: track 9.75 -> 6.03 mm
- net /D26DAC2: track 83.8 -> 86.4 mm
- net /Vout7: track 37.4 -> 39.1 mm
- removed copper zone on B.Cu, net +3.3VADC
Other:
- board text added: "+"
- board text added: "-"
- board text added: "12V"
- board text added: "5V"
- board text added: "9V"
- board text added: "CH0-PIN12"
- board text added: "CH0-PIN13"
- board text added: "CH0-PIN14"
- board text added: "CH0-PIN27"
- board text added: "CH0-PIN33"
