File: hardware/kicad/reactor/reactor.kicad_sch (KiCad schematic)
At the start: 28 parts, among them J1 Conn_01x02_Pin, J2 Conn_01x02_Pin, J3 Conn_01x02_Pin, J4 Conn_02x09_Odd_Even, J5 Conn_01x02_Pin, J6 Conn_01x10, J7 Conn_01x03, U1 LD1117S50TR, U2 LD1117S33TR, U3 LD1117S33TR

Commit message: bug fix; reactor board update;
Parts:
- removed C1, C3, C5: 0.1uF, Capacitor_SMD:CP_Elec_4x5.4, symbol Device:C_Polarized
- removed C2, C4, C6: 10uF, Capacitor_SMD:CP_Elec_4x5.3, symbol Device:C_Polarized
- removed U2, U3: LD1117S33TR, Package_TO_SOT_SMD:SOT-223-3_TabPin2, symbol Regulator_Linear:LD1117S33TR_SOT223
- added C1: 0.22uF, Capacitor_SMD:C_0805_2012Metric_Pad1.18x1.45mm_HandSolder, symbol Device:C
- added C2, C3, C4, C5, C6: 0.1uF, Capacitor_SMD:C_1206_3216Metric, symbol Device:C
- added D4, D5: 50V 5A, Diode_SMD:D_SMA, symbol Diode:1N5817
- added U2, U3: TLV75733PDBV, Package_TO_SOT_SMD:SOT-23-5, symbol Regulator_Linear:TLV75733PDBV
- U1: value LD1117S50TR -> LM340MPX-5.0/NOPB
Connections:
- net +12V: now also J3.2 (Pin_2); no longer J3.1 (Pin_1)
- net +3.3V: now also C4.1, D4.2 (A), U2.5 (OUT)
- net +3.3VADC: now also C6.1, D5.2 (A), U3.5 (OUT)
- net +5V: now also C2.1, C3.1, C5.1, D4.1 (K), D5.1 (K), U2.1 (IN), U2.3 (EN), U3.1 (IN), U3.3 (EN)
- net GND: now also C1.2, C2.2, C3.2, C4.2, C5.2, C6.2, U2.2 (GND), U3.2 (GND)
- net GNDPWR: now also J3.1 (Pin_1); no longer J3.2 (Pin_2)
- net Vcc_protected: now also C1.1
Other:
- moved on the sheet: J1, J3
