File: hardware/kicad/turbidometer/turbidometer.kicad_pcb (KiCad board)
At the start: 2 copper layers, 80 x 70 mm, 56 parts, among them J1 Conn_01x04, J2 Conn_01x02_Pin, J3 Conn_01x02_Pin, J4 Conn_01x03_Pin, J5 Conn_01x04, J6 Conn_01x04, J7 Conn_01x02_Pin, Q1 IRLML6344TRPBF, Q2 IRLML6344TRPBF, Q3 IRLML6344TRPBF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

Commit message: bug fix; reactor board update;
Parts:
- removed Vbias: TestPoint, TestPoint:TestPoint_Pad_1.0x1.0mm
- added R17: 10K, Resistor_SMD:R_0805_2012Metric_Pad1.20x1.40mm_HandSolder, F.Cu at (131.0, 61.2)
- added R18: 10K, Resistor_SMD:R_0805_2012Metric_Pad1.20x1.40mm_HandSolder, F.Cu at (132.0, 73.3)
- added R19: 10K, Resistor_SMD:R_0805_2012Metric_Pad1.20x1.40mm_HandSolder, F.Cu at (130.6, 86.0)
- added Vbias1: TestPoint, TestPoint:TestPoint_Pad_1.0x1.0mm, F.Cu at (139.9, 97.8)
- R11: value R_US -> 45K
- R12: value R_US -> 1M
- moved J3 10.4 mm to (129.0, 46.5)
- moved J1 8.75 mm to (129.1, 94.5)
- moved R10 8.75 mm to (135.4, 98.8)
- moved R9 8.75 mm to (135.4, 94.7)
- moved TP2 8.66 mm to (129.2, 91.0)
- moved TP1 6.73 mm to (134.9, 46.4)
- moved R13 5.53 mm to (130.7, 83.2), turned to 180 degrees
- moved VREF2 5.13 mm to (131.6, 80.3)
- moved U7 4.92 mm to (135.4, 83.8)
- moved LED2 4.92 mm to (146.7, 92.0)
- moved C13 4.65 mm to (138.7, 85.5)
- moved C14 4.52 mm to (137.5, 80.6)
- moved R15 4.51 mm to (142.2, 86.7)
- moved R1 4.42 mm to (131.0, 58.1), turned to 180 degrees
- moved R16 4.41 mm to (147.7, 89.0)
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Routing:
- net /LED_NEG1: track 6.00 -> 79.1 mm
- net /LED_NEG2: track 15.9 -> 88.7 mm
- net /LED_NEG0: track 2.13 -> 73.5 mm
- net /Vbias: track 6.69 -> 68.9 mm
- net +5V: track 89.8 -> 150.1 mm
- net /A1: track 12.6 -> 65.6 mm
- net +3.3V: track 43.8 -> 87.3 mm
- net /A0: track 11.1 -> 38.6 mm
- net /PD_FB1: track 11.5 -> 20.3 mm
- net /PD_FB0: track 15.0 -> 19.6 mm
- net Net-(U3-+): track 4.97 -> 9.26 mm
- net Net-(U7-+): track 4.66 -> 8.61 mm
- net Net-(U4-+): track 4.77 -> 8.60 mm
- net /VREF1: track 6.87 -> 3.34 mm
- net /LED_SENS2: track 7.01 -> 9.19 mm
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