File: hardware/kicad/turbidometer/turbidometer.kicad_sch (KiCad schematic)
At the start: 56 parts, among them J1 Conn_01x04, J2 Conn_01x02_Pin, J3 Conn_01x02_Pin, J4 Conn_01x03_Pin, J5 Conn_01x04, J6 Conn_01x04, J7 Conn_01x02_Pin, Q1 IRLML6344TRPBF, Q2 IRLML6344TRPBF, Q3 IRLML6344TRPBF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

Commit message: bug fix; reactor board update;
Parts:
- added R17, R18, R19: 10K, Resistor_SMD:R_0805_2012Metric_Pad1.20x1.40mm_HandSolder, symbol Device:R_US
- R11: value R_US -> 45K
- R12: value R_US -> 1M
Connections:
- net GND: now also R17.2, R18.2, R19.2
- net at R1.1, U3.1 (+), VREF0.1: now also R17.1
- net at R5.1, U4.1 (+), VREF1.1: now also R18.1
- net at R13.1, U7.1 (+), VREF2.1: now also R19.1
